File: 1wireESP.brd (EAGLE design)
At the start: 15.9 x 15.2 mm, 16 parts

Commit message: smd
Connections:
- removed net N$6: 02.TP, U$2.GPIO02
- new net N$3: 02.TP, U$2.GPIO16
- net N$4: now also U$2.GPIO02; no longer U$2.GPIO16
Routing:
- net N$4: track 8.05 -> 18.0 mm
- net N$3: track 0.00 -> 9.91 mm
- net N$6: track 5.74 -> 0.00 mm
- net GND: track 3.85 -> 0.00 mm, vias 9 -> 0
- net +5V: track 13.3 -> 11.4 mm
- net N$1: track 5.98 -> 5.84 mm, vias 0 -> 1
