File: ESPRGBLED.sch (EAGLE design)
At the start: 5 parts

Commit message: added layout
Parts:
- removed D4: (no value), diode:DIODE-SMB
- removed SV1: (no value), con-lstb:MA03-1
- added C1, C2: (no value), rcl:C-EUC0603K
- added C3, C4: (no value), rcl:C-EUC0805K
- added D1: MBRS130LT3, diode:MBRS130LT3
- added U$3: (no value), Fabian:3-WIRE_CONNWIRE
- added U$4, U$5, U$6, U$7, U$8: CON1, Fabian:CON1
Connections:
- new net N$1: U$4.P$1
- new net N$4: U$5.P$1
- new net N$5: U$6.P$1
- new net OUT: D1.A
- new net SUPP: D1.C
- net +12V: now also C1.1, C3.1, D1.C, U$7.P$1; no longer D4.C
- net GND: now also C1.2, C2.2, C3.2, C4.2, D1.A, U$3.0V, U$8.P$1; no longer D4.A, SV1.1
- net N$7: now also U$3.SIG; no longer SV1.3
- net N$8: now also U$3.5V; no longer SV1.2
- net VCC: now also C2.1, C4.1

Commit message: layouted
Parts:
- added R1: 0R, rcl:R-EU_R0603
- added U$9: CON1, Fabian:CON1
Connections:
- new net DGND: C1.2, C2.2, C3.2, C4.2, R1.1, U$1.GND, U$2.GND, U$2.GPIO15, U$3.0V
- new net N$2: U$2.GPIO13
- net +12V: now also U$9.P$1
- net GND: now also R1.2; no longer C1.2, C2.2, C3.2, C4.2, U$1.GND, U$2.GND, U$2.GPIO15, U$3.0V

Commit message: updated layouts
Parts:
- added R2: 0R, rcl:R-EU_R0603
- C1, C2: MF (none) -> AVX; MPN (none) -> 0603YC104K4T4A; OC_FARNELL (none) -> 1833863
- C3, C4: MF (none) -> AVX; MPN (none) -> 08055C224KAZ2A; OC_FARNELL (none) -> 2332797
- D1: MF (none) -> ON SEMICONDUCTOR; MPN (none) -> MBRS130LT3G; OC_FARNELL (none) -> 2125539
- R1: MF (none) -> BOURNS; MPN (none) -> CR0603-J/-000ELF; OC_FARNELL (none) -> 2467553
- R5: MF (none) -> WELWYN; MPN (none) -> ASC0603-10KFT5; OC_FARNELL (none) -> 2078915RL
- U$1: MF (none) -> STMICROELECTRONICS; MPN (none) -> LD1117S33TR; OC_FARNELL (none) -> 1202826
- U$2, U$3, U$4, U$5, U$6, U$7, U$8, U$9: OC_FARNELL (none) -> unknown
Connections:
- new net N$9: R2.1, U$2.GPIO0
- net DGND: now also R2.2

Commit message: smd
Parts:
- removed U$2: ESP8266, ESP8266:ESP8266
- added MDL1: (no value), ESP8266-ESP12E:ESP8266-12EESP8266-ESP12E
- added R3: 100k, rcl:R-EU_R0603
- added R4: 10k, rcl:R-EU_R0603
- R2: device rcl:R-EU_R0603 -> rcl:R-EU_R0805
Connections:
- new net N$10: MDL1.ADC, R3.1, R4.2
- net +12V: now also R3.2
- net DGND: now also MDL1.GND, MDL1.GPIO15; no longer U$2.GND, U$2.GPIO15
- net GND: now also R4.1
- net N$11: now also MDL1.CH_PD; no longer U$2.CH_PD
- net N$2: now also MDL1.GPIO14; no longer U$2.GPIO13
- net N$3: now also MDL1.GPIO12; no longer U$2.GPIO12
- net N$6: now also MDL1.GPIO13; no longer U$2.GPIO14
- net N$7: now also MDL1.RXD; no longer U$2.URXD
- net N$8: now also MDL1.TXD; no longer U$2.UTXD
- net N$9: now also MDL1.GPIO0; no longer U$2.GPIO0
- net VCC: now also MDL1.VCC; no longer U$2.VCC
Other:
- moved on the sheet: R2, R5

Commit message: through hole
Parts:
- removed U$4, U$5, U$6, U$7, U$8, U$9: CON1, Fabian:CON1
- added LSP1, LSP2, LSP3, LSP4, LSP5, LSP6: LSP10, solpad:LSP10
Connections:
- net +12V: now also LSP1.MP, LSP5.MP; no longer U$7.P$1, U$9.P$1
- net DGND: now also R4.1
- net GND: now also LSP6.MP; no longer R4.1, U$8.P$1
- net N$1: now also LSP2.MP; no longer U$4.P$1
- net N$4: now also LSP3.MP; no longer U$5.P$1
- net N$5: now also LSP4.MP; no longer U$6.P$1
Changed lines of the file:
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@@
-<attribute name="OC_FARNELL" value="unknown"/>
-</part>
-<part name="U$4" library="Fabian" deviceset="CON1" device="">
-<attribute name="MF" value=""/>
-<attribute name="MPN" value=""/>
-<attribute name="OC_FARNELL" value="unknown"/>
-</part>
-<part name="U$5" library="Fabian" deviceset="CON1" device="">
-<attribute name="MF" value=""/>
-<attribute name="MPN" value=""/>
-<attribute name="OC_FARNELL" value="unknown"/>
-</part>
-<part name="U$6" library="Fabian" deviceset="CON1" device="">
-<attribute name="MF" value=""/>
-<attribute name="MPN" value=""/>
-<attribute name="OC_FARNELL" value="unknown"/>
-</part>
-<part name="U$7" library="Fabian" deviceset="CON1" device="">
-<attribute name="MF" value=""/>
-<attribute name="MPN" value=""/>
-<attribute name="OC_FARNELL" value="unknown"/>
-</part>
-<part name="U$8" library="Fabian" deviceset="CON1" device="">
-<attribute name="MF" value=""/>
-<attribute name="MPN" value=""/>
 <attribute name="OC_FARNELL" value="unknown"/>
 </part>
 <part name="SUPPLY9" library="supply2" deviceset="+12V" device=""/>
 <part name="GND12" library="supply1" deviceset="GND" device=""/>
-<part name="U$9" library="Fabian" deviceset="CON1" device="">
-<attribute name="MF" value=""/>
-<attribute name="MPN" value=""/>
-<attribute name="OC_FARNELL" value="unknown"/>
-</part>
 <part name="SUPPLY10" library="supply2" deviceset="+12V" device=""/>
 <part name="SUPPLY11" library="supply2" deviceset="DGND" device=""/>
@@
 </part>
 <part name="SUPPLY12" library="supply2" deviceset="+12V" device=""/>
-<part name="GND4" library="supply1" deviceset="GND" device=""/>
+<part name="LSP1" library="solpad" deviceset="LSP10" device=""/>
+<part name="LSP2" library="solpad" deviceset="LSP10" device=""/>
+<part name="LSP3" library="solpad" deviceset="LSP10" device=""/>
+<part name="LSP4" library="solpad" deviceset="LSP10" device=""/>
+<part name="LSP5" library="solpad" deviceset="LSP10" device=""/>
+<part name="LSP6" library="solpad" deviceset="LSP10" device=""/>
+<part name="SUPPLY20" library="supply2" deviceset="DGND" device=""/>
 </parts>
 <sheets>
@@
 <attribute name="MPN" x="0" y="48.26" size="1.778" layer="96" display="off"/>
 </instance>
-<instance part="U$4" gate="G$1" x="162.56" y="149.86">
-<attribute name="OC_FARNELL" x="162.56" y="149.86" size="1.778" layer="96" display="off"/>
-<attribute name="MF" x="162.56" y="149.86" size="1.778" layer="96" display="off"/>
-<attribute name="MPN" x="162.56" y="149.86" size="1.778" layer="96" display="off"/>
-</instance>
-<instance part="U$5" gate="G$1" x="154.94" y="96.52">
-<attribute name="OC_FARNELL" x="154.94" y="96.52" size="1.778" layer="96" display="off"/>
-<attribute name="MF" x="154.94" y="96.52" size="1.778" layer="96" display="off"/>
-<attribute name="MPN" x="154.94" y="96.52" size="1.778" layer="96" display="off"/>
-</instance>
-<instance part="U$6" gate="G$1" x="154.94" y="45.72">
-<attribute name="OC_FARNELL" x="154.94" y="45.72" size="1.778" layer="96" display="off"/>
-<attribute name="MF" x="154.94" y="45.72" size="1.778" layer="96" display="off"/>
-<attribute name="MPN" x="154.94" y="45.72" size="1.778" layer="96" display="off"/>
-</instance>
-<instance part="U$7" gate="G$1" x="2.54" y="147.32">
-<attribute name="OC_FARNELL" x="2.54" y="147.32" size="1.778" layer="96" display="off"/>
-<attribute name="MF" x="2.54" y="147.32" size="1.778" layer="96" display="off"/>
-<attribute name="MPN" x="2.54" y="147.32" size="1.778" layer="96" display="off"/>
-</instance>
-<instance part="U$8" gate="G$1" x="2.54" y="137.16">
-<attribute name="OC_FARNELL" x="2.54" y="137.16" size="1.778" layer="96" display="off"/>
-<attribute name="MF" x="2.54" y="137.16" size="1.778" layer="96" display="off"/>
-<attribute name="MPN" x="2.54" y="137.16" size="1.778" layer="96" display="off"/>
-</instance>
 <instance part="SUPPLY9" gate="+12V" x="0" y="149.86"/>
 <instance part="GND12" gate="1" x="0" y="134.62"/>
-<instance part="U$9" gate="G$1" x="160.02" y="162.56">
-<attribute name="OC_FARNELL" x="160.02" y="162.56" size="1.778" layer="96" display="off"/>
-<attribute name="MF" x="160.02" y="162.56" size="1.778" layer="96" display="off"/>
-<attribute name="MPN" x="160.02" y="162.56" size="1.778" layer="96" display="off"/>
-</instance>
 <instance part="SUPPLY10" gate="+12V" x="157.48" y="165.1"/>
 <instance part="SUPPLY11" gate="G$1" x="17.78" y="20.32"/>
@@
 </instance>
 <instance part="SUPPLY12" gate="+12V" x="96.52" y="43.18"/>
-<instance part="GND4" gate="1" x="96.52" y="7.62"/>
+<instance part="LSP1" gate="1" x="172.72" y="162.56" rot="R270"/>
+<instance part="LSP2" gate="1" x="172.72" y="149.86" rot="R270"/>
+<instance part="LSP3" gate="1" x="172.72" y="96.52" rot="R270"/>
+<instance part="LSP4" gate="1" x="175.26" y="45.72" rot="R270"/>
+<instance part="LSP5" gate="1" x="22.86" y="147.32" rot="R270"/>
+<instance part="LSP6" gate="1" x="22.86" y="137.16" rot="R270"/>
+<instance part="SUPPLY20" gate="G$1" x="96.52" y="7.62"/>
 </instances>
 <busses>
@@
 </segment>
 <segment>
-<pinref part="U$7" gate="G$1" pin="P$1"/>
 <pinref part="SUPPLY9" gate="+12V" pin="+12V"/>
-</segment>
-<segment>
-<pinref part="U$9" gate="G$1" pin="P$1"/>
+<wire x1="20.32" y1="147.32" x2="0" y2="147.32" width="0.1524" layer="91"/>
+<pinref part="LSP5" gate="1" pin="MP"/>
+</segment>
+<segment>
 <pinref part="SUPPLY10" gate="+12V" pin="+12V"/>
+<wire x1="170.18" y1="162.56" x2="157.48" y2="162.56" width="0.1524" layer="91"/>
+<pinref part="LSP1" gate="1" pin="MP"/>
 </segment>
 <segment>
@@
 </segment>
 <segment>
-<pinref part="U$8" gate="G$1" pin="P$1"/>
 <pinref part="GND12" gate="1" pin="GND"/>
+<wire x1="20.32" y1="137.16" x2="0" y2="137.16" width="0.1524" layer="91"/>
+<pinref part="LSP6" gate="1" pin="MP"/>
 </segment>
 <segment>
@@
 <pinref part="R1" gate="G$1" pin="2"/>
 <wire x1="2.54" y1="27.94" x2="5.08" y2="27.94" width="0.1524" layer="91"/>
-</segment>
-<segment>
-<pinref part="R4" gate="G$1" pin="1"/>
-<pinref part="GND4" gate="1" pin="GND"/>
-<wire x1="96.52" y1="12.7" x2="96.52" y2="10.16" width="0.1524" layer="91"/>
 </segment>
 </net>
@@
 <segment>
 <portref moduleinst="PWR1" port="OUT"/>
-<pinref part="U$4" gate="G$1" pin="P$1"/>
-<wire x1="160.02" y1="149.86" x2="152.4" y2="149.86" width="0.1524" layer="91"/>
+<wire x1="170.18" y1="149.86" x2="152.4" y2="149.86" width="0.1524" layer="91"/>
+<pinref part="LSP2" gate="1" pin="MP"/>
 </segment>
 </net>
@@
 <segment>
 <portref moduleinst="PWR2" port="OUT"/>
-<pinref part="U$5" gate="G$1" pin="P$1"/>
+<wire x1="170.18" y1="96.52" x2="152.4" y2="96.52" width="0.1524" layer="91"/>
+<pinref part="LSP3" gate="1" pin="MP"/>
 </segment>
 </net>
@@
 <segment>
 <portref moduleinst="PWR3" port="OUT"/>
-<pinref part="U$6" gate="G$1" pin="P$1"/>
+<wire x1="172.72" y1="45.72" x2="152.4" y2="45.72" width="0.1524" layer="91"/>
+<pinref part="LSP4" gate="1" pin="MP"/>
 </segment>
 </net>
@@
 <wire x1="17.78" y1="27.94" x2="17.78" y2="22.86" width="0.1524" layer="91"/>
 </segment>
-</net>
+<segment>
+<pinref part="R4" gate="G$1" pin="1"/>
+<wire x1="96.52" y1="12.7" x2="96.52" y2="10.16" width="0.1524" layer="91"/>
+<pinref part="SUPPLY20" gate="G$1" pin="DGND"/>
+</segment>
+</net>

Commit message: minor stuff
Parts:
- renumbered LSP1 to +, LSP2 to 13, LSP3 to 12, LSP4 to 14, LSP5 to 12V, LSP6 to GND
Changed lines of the file:
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@@
 <grid distance="0.1" unitdist="inch" unit="inch" style="lines" multiple="1" display="no" altdistance="0.01" altunitdist="inch" altunit="inch"/>
 <layers>
-<layer number="1" name="Top" color="4" fill="1" visible="yes" active="no"/>
-<layer number="2" name="Route2" color="1" fill="3" visible="yes" active="no"/>
-<layer number="3" name="Route3" color="4" fill="3" visible="yes" active="no"/>
-<layer number="14" name="Route14" color="1" fill="6" visible="yes" active="no"/>
-<layer number="15" name="Route15" color="4" fill="6" visible="yes" active="no"/>
-<layer number="16" name="Bottom" color="1" fill="1" visible="yes" active="no"/>
-<layer number="17" name="Pads" color="2" fill="1" visible="yes" active="no"/>
-<layer number="18" name="Vias" color="2" fill="1" visible="yes" active="no"/>
-<layer number="19" name="Unrouted" color="6" fill="1" visible="yes" active="no"/>
-<layer number="20" name="Dimension" color="15" fill="1" visible="yes" active="no"/>
-<layer number="21" name="tPlace" color="7" fill="1" visible="yes" active="no"/>
-<layer number="22" name="bPlace" color="7" fill="1" visible="yes" active="no"/>
-<layer number="23" name="tOrigins" color="15" fill="1" visible="yes" active="no"/>
-<layer number="24" name="bOrigins" color="15" fill="1" visible="yes" active="no"/>
-<layer number="25" name="tNames" color="7" fill="1" visible="yes" active="no"/>
-<layer number="26" name="bNames" color="7" fill="1" visible="yes" active="no"/>
-<layer number="27" name="tValues" color="7" fill="1" visible="yes" active="no"/>
-<layer number="28" name="bValues" color="7" fill="1" visible="yes" active="no"/>
+<layer number="1" name="Top" color="4" fill="1" visible="no" active="no"/>
+<layer number="2" name="Route2" color="1" fill="3" visible="no" active="no"/>
+<layer number="3" name="Route3" color="4" fill="3" visible="no" active="no"/>
+<layer number="14" name="Route14" color="1" fill="6" visible="no" active="no"/>
+<layer number="15" name="Route15" color="4" fill="6" visible="no" active="no"/>
+<layer number="16" name="Bottom" color="1" fill="1" visible="no" active="no"/>
+<layer number="17" name="Pads" color="2" fill="1" visible="no" active="no"/>
+<layer number="18" name="Vias" color="2" fill="1" visible="no" active="no"/>
+<layer number="19" name="Unrouted" color="6" fill="1" visible="no" active="no"/>
+<layer number="20" name="Dimension" color="15" fill="1" visible="no" active="no"/>
+<layer number="21" name="tPlace" color="7" fill="1" visible="no" active="no"/>
+<layer number="22" name="bPlace" color="7" fill="1" visible="no" active="no"/>
+<layer number="23" name="tOrigins" color="15" fill="1" visible="no" active="no"/>
+<layer number="24" name="bOrigins" color="15" fill="1" visible="no" active="no"/>
+<layer number="25" name="tNames" color="7" fill="1" visible="no" active="no"/>
+<layer number="26" name="bNames" color="7" fill="1" visible="no" active="no"/>
+<layer number="27" name="tValues" color="7" fill="1" visible="no" active="no"/>
+<layer number="28" name="bValues" color="7" fill="1" visible="no" active="no"/>
 <layer number="29" name="tStop" color="7" fill="3" visible="no" active="no"/>
 <layer number="30" name="bStop" color="7" fill="6" visible="no" active="no"/>
@@
 <layer number="35" name="tGlue" color="7" fill="4" visible="no" active="no"/>
 <layer number="36" name="bGlue" color="7" fill="5" visible="no" active="no"/>
-<layer number="37" name="tTest" color="7" fill="1" visible="yes" active="no"/>
-<layer number="38" name="bTest" color="7" fill="1" visible="yes" active="no"/>
+<layer number="37" name="tTest" color="7" fill="1" visible="no" active="no"/>
+<layer number="38" name="bTest" color="7" fill="1" visible="no" active="no"/>
 <layer number="39" name="tKeepout" color="4" fill="11" visible="no" active="no"/>
 <layer number="40" name="bKeepout" color="1" fill="11" visible="no" active="no"/>
@@
 <layer number="44" name="Drills" color="7" fill="1" visible="no" active="no"/>
 <layer number="45" name="Holes" color="7" fill="1" visible="no" active="no"/>
-<layer number="46" name="Milling" color="3" fill="1" visible="yes" active="no"/>
-<layer number="47" name="Measures" color="7" fill="1" visible="yes" active="no"/>
-<layer number="48" name="Document" color="7" fill="1" visible="yes" active="no"/>
-<layer number="49" name="Reference" color="7" fill="1" visible="yes" active="no"/>
-<layer number="50" name="dxf" color="7" fill="1" visible="yes" active="no"/>
-<layer number="51" name="tDocu" color="7" fill="1" visible="yes" active="no"/>
-<layer number="52" name="bDocu" color="7" fill="1" visible="yes" active="no"/>
-<layer number="53" name="tGND_GNDA" color="7" fill="1" visible="yes" active="no"/>
-<layer number="54" name="bGND_GNDA" color="7" fill="1" visible="yes" active="no"/>
-<layer number="56" name="wert" color="7" fill="1" visible="yes" active="no"/>
+<layer number="46" name="Milling" color="3" fill="1" visible="no" active="no"/>
+<layer number="47" name="Measures" color="7" fill="1" visible="no" active="no"/>
+<layer number="48" name="Document" color="7" fill="1" visible="no" active="no"/>
+<layer number="49" name="Reference" color="7" fill="1" visible="no" active="no"/>
+<layer number="50" name="dxf" color="7" fill="1" visible="no" active="no"/>
+<layer number="51" name="tDocu" color="7" fill="1" visible="no" active="no"/>
+<layer number="52" name="bDocu" color="7" fill="1" visible="no" active="no"/>
+<layer number="53" name="tGND_GNDA" color="7" fill="1" visible="no" active="no"/>
+<layer number="54" name="bGND_GNDA" color="7" fill="1" visible="no" active="no"/>
+<layer number="56" name="wert" color="7" fill="1" visible="no" active="no"/>
 <layer number="90" name="Modules" color="5" fill="1" visible="yes" active="yes"/>
 <layer number="91" name="Nets" color="2" fill="1" visible="yes" active="yes"/>
@@
 </part>
 <part name="SUPPLY12" library="supply2" deviceset="+12V" device=""/>
-<part name="LSP1" library="solpad" deviceset="LSP10" device=""/>
-<part name="LSP2" library="solpad" deviceset="LSP10" device=""/>
-<part name="LSP3" library="solpad" deviceset="LSP10" device=""/>
-<part name="LSP4" library="solpad" deviceset="LSP10" device=""/>
-<part name="LSP5" library="solpad" deviceset="LSP10" device=""/>
-<part name="LSP6" library="solpad" deviceset="LSP10" device=""/>
+<part name="+" library="solpad" deviceset="LSP10" device=""/>
+<part name="13" library="solpad" deviceset="LSP10" device=""/>
+<part name="12" library="solpad" deviceset="LSP10" device=""/>
+<part name="14" library="solpad" deviceset="LSP10" device=""/>
+<part name="12V" library="solpad" deviceset="LSP10" device=""/>
+<part name="GND" library="solpad" deviceset="LSP10" device=""/>
 <part name="SUPPLY20" library="supply2" deviceset="DGND" device=""/>
 </parts>
@@
 </instance>
 <instance part="SUPPLY12" gate="+12V" x="96.52" y="43.18"/>
-<instance part="LSP1" gate="1" x="172.72" y="162.56" rot="R270"/>
-<instance part="LSP2" gate="1" x="172.72" y="149.86" rot="R270"/>
-<instance part="LSP3" gate="1" x="172.72" y="96.52" rot="R270"/>
-<instance part="LSP4" gate="1" x="175.26" y="45.72" rot="R270"/>
-<instance part="LSP5" gate="1" x="22.86" y="147.32" rot="R270"/>
-<instance part="LSP6" gate="1" x="22.86" y="137.16" rot="R270"/>
+<instance part="+" gate="1" x="172.72" y="162.56" rot="R270"/>
+<instance part="13" gate="1" x="172.72" y="149.86" rot="R270"/>
+<instance part="12" gate="1" x="172.72" y="96.52" rot="R270"/>
+<instance part="14" gate="1" x="175.26" y="45.72" rot="R270"/>
+<instance part="12V" gate="1" x="22.86" y="147.32" rot="R270"/>
+<instance part="GND" gate="1" x="22.86" y="137.16" rot="R270"/>
 <instance part="SUPPLY20" gate="G$1" x="96.52" y="7.62"/>
 </instances>
@@
 <pinref part="SUPPLY9" gate="+12V" pin="+12V"/>
 <wire x1="20.32" y1="147.32" x2="0" y2="147.32" width="0.1524" layer="91"/>
-<pinref part="LSP5" gate="1" pin="MP"/>
+<pinref part="12V" gate="1" pin="MP"/>
 </segment>
 <segment>
 <pinref part="SUPPLY10" gate="+12V" pin="+12V"/>
 <wire x1="170.18" y1="162.56" x2="157.48" y2="162.56" width="0.1524" layer="91"/>
-<pinref part="LSP1" gate="1" pin="MP"/>
+<pinref part="+" gate="1" pin="MP"/>
 </segment>
 <segment>
@@
 <pinref part="GND12" gate="1" pin="GND"/>
 <wire x1="20.32" y1="137.16" x2="0" y2="137.16" width="0.1524" layer="91"/>
-<pinref part="LSP6" gate="1" pin="MP"/>
+<pinref part="GND" gate="1" pin="MP"/>
 </segment>
 <segment>
@@
 <portref moduleinst="PWR1" port="OUT"/>
 <wire x1="170.18" y1="149.86" x2="152.4" y2="149.86" width="0.1524" layer="91"/>
-<pinref part="LSP2" gate="1" pin="MP"/>
+<pinref part="13" gate="1" pin="MP"/>
 </segment>
 </net>
@@
 <portref moduleinst="PWR2" port="OUT"/>
 <wire x1="170.18" y1="96.52" x2="152.4" y2="96.52" width="0.1524" layer="91"/>
-<pinref part="LSP3" gate="1" pin="MP"/>
+<pinref part="12" gate="1" pin="MP"/>
 </segment>
 </net>
@@
 <portref moduleinst="PWR3" port="OUT"/>
 <wire x1="172.72" y1="45.72" x2="152.4" y2="45.72" width="0.1524" layer="91"/>
-<pinref part="LSP4" gate="1" pin="MP"/>
-</segment>
-</net>
+<pinref part="14" gate="1" pin="MP"/>
+</segment>
+</net>

Commit message: updated HW with reset-wakeup option
Parts:
- removed R5: 10k, rcl:R-EU_R0603
- added JMP1: 0R-JUMPC, jump-0r-smd:0R-JUMPC
Connections:
- new net N$12: JMP1-0R.2, MDL1.CH_PD
- net N$11: now also JMP1-0R.1, MDL1.REST; no longer MDL1.CH_PD, R5.1
- net VCC: now also JMP1-0R.3; no longer R5.2
Changed lines of the file:
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@@
 <part name="SUPPLY6" library="supply2" deviceset="+12V" device=""/>
 <part name="GND7" library="supply1" deviceset="GND" device=""/>
-<part name="R5" library="rcl" deviceset="R-EU_" device="R0603" value="10k">
-<attribute name="MF" value="WELWYN"/>
-<attribute name="MPN" value="ASC0603-10KFT5"/>
-<attribute name="OC_FARNELL" value="2078915RL"/>
-</part>
 <part name="SUPPLY7" library="supply2" deviceset="VCC" device=""/>
 <part name="SUPPLY1" library="supply2" deviceset="+12V" device=""/>
@@
 <part name="GND" library="solpad" deviceset="LSP10" device=""/>
 <part name="SUPPLY20" library="supply2" deviceset="DGND" device=""/>
+<part name="JMP1" library="jump-0r-smd" deviceset="0R-JUMP" device="C"/>
 </parts>
 <sheets>
@@
 <instance part="SUPPLY6" gate="+12V" x="-45.72" y="139.7"/>
 <instance part="GND7" gate="1" x="-45.72" y="96.52"/>
-<instance part="R5" gate="G$1" x="96.52" y="76.2" rot="R90">
-<attribute name="OC_FARNELL" x="96.52" y="76.2" size="1.778" layer="96" display="off"/>
-<attribute name="MF" x="96.52" y="76.2" size="1.778" layer="96" display="off"/>
-<attribute name="MPN" x="96.52" y="76.2" size="1.778" layer="96" display="off"/>
-</instance>
 <instance part="SUPPLY7" gate="G$1" x="96.52" y="91.44"/>
 <instance part="SUPPLY1" gate="+12V" x="132.08" y="109.22"/>
@@
 <instance part="GND" gate="1" x="22.86" y="137.16" rot="R270"/>
 <instance part="SUPPLY20" gate="G$1" x="96.52" y="7.62"/>
+<instance part="JMP1" gate="-0R" x="91.44" y="53.34" rot="R180"/>
+<instance part="JMP1" gate="G$2" x="93.98" y="50.8" rot="R180"/>
 </instances>
 <busses>
@@
 </segment>
 <segment>
-<pinref part="R5" gate="G$1" pin="2"/>
 <pinref part="SUPPLY7" gate="G$1" pin="VCC"/>
 <wire x1="96.52" y1="88.9" x2="96.52" y2="81.28" width="0.1524" layer="91"/>
+<wire x1="96.52" y1="81.28" x2="96.52" y2="71.12" width="0.1524" layer="91"/>
+<pinref part="JMP1" gate="-0R" pin="3"/>
+<wire x1="96.52" y1="71.12" x2="91.44" y2="71.12" width="0.1524" layer="91"/>
+<wire x1="91.44" y1="71.12" x2="91.44" y2="55.88" width="0.1524" layer="91"/>
 </segment>
 </net>
@@
 <pinref part="U$3" gate="G$1" pin="5V"/>
 <pinref part="MDL1" gate="G$1" pin="TXD"/>
-</segment>
-</net>
-<net name="N$11" class="0">
-<segment>
-<pinref part="R5" gate="G$1" pin="1"/>
-<wire x1="96.52" y1="71.12" x2="96.52" y2="55.88" width="0.1524" layer="91"/>
-<wire x1="96.52" y1="55.88" x2="96.52" y2="53.34" width="0.1524" layer="91"/>
-<wire x1="96.52" y1="53.34" x2="81.28" y2="53.34" width="0.1524" layer="91"/>
-<pinref part="MDL1" gate="G$1" pin="CH_PD"/>
 </segment>
 </net>
@@
 </segment>
 </net>
+<net name="N$12" class="0">
+<segment>
+<pinref part="MDL1" gate="G$1" pin="CH_PD"/>
+<pinref part="JMP1" gate="-0R" pin="2"/>
+<wire x1="88.9" y1="53.34" x2="81.28" y2="53.34" width="0.1524" layer="91"/>
+</segment>
+</net>
+<net name="N$11" class="0">
+<segment>
+<pinref part="JMP1" gate="-0R" pin="1"/>
+<wire x1="91.44" y1="50.8" x2="91.44" y2="48.26" width="0.1524" layer="91"/>
+<pinref part="MDL1" gate="G$1" pin="REST"/>
+<wire x1="91.44" y1="48.26" x2="81.28" y2="48.26" width="0.1524" layer="91"/>
+</segment>
+</net>
