File: ESPRGBLED.sch (EAGLE design)
At the start: 18 parts

Commit message: superminiaturized
Parts:
- added C1, C2: 10uF, rcl:C-EUC0805K
- added R1: 0R, rcl:R-EU_R0402
- R5: value (none) -> 61k9
- R6: value (none) -> 20k
Connections:
- net N$10 renamed ADC
- net N$11 renamed REST
- net N$12 renamed CH_PD
- net N$2 renamed GPIO14
- net N$3 renamed GPIO12
- net N$6 renamed GPIO13
- net N$9 renamed GPIO0
- new net VIN: C1.1, C2.1, R1.2, R3.2, U$2.VIN
- net +12V: now also R1.1; no longer R3.2, U$2.VIN
- net GND: now also C1.2, C2.2
Other:
- moved on the sheet: JMP1-0R
